File: board/kicad/HG1-ANT.kicad_pcb (KiCad board)
At the start: 10 copper layers, 150 x 190 mm, 67 parts, among them J1 Molex Micro-Fit 4p: +28V_PA, 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, J2 Samtec LSHM-150 JESD204B x12 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, J3 Samtec LSHM-150 JESD204B x12 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, J4 Samtec LSHM-120 SPI/sync/GNSS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, U1 ADF4159 FMCW PLL (TX chirp), U10 HRX-8 8-ch Ku SiGe RX RFIC (L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, U11 HRX-8 8-ch Ku SiGe RX RFIC (L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, U12 HRX-8 8-ch Ku SiGe RX RFIC (L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, U13 HRX-8 8-ch Ku SiGe RX RFIC (L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, U14 HRX-8 8-ch Ku SiGe RX RFIC (L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, U15 HRX-8 8-ch Ku SiGe RX RFIC (L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, U2 HMC733 VCO 10-20 GHz (TX), U20 AD9083BBCZ 16-ch 125 MHz CTSD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, U21 AD9083BBCZ 16-ch 125 MHz CTSD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, U22 AD9083BBCZ 16-ch 125 MHz CTSD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, U23 AD9083BBCZ 16-ch 125 MHz CTSD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, U24 AD9083BBCZ 16-ch 125 MHz CTSD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, U25 AD9083BBCZ 16-ch 125 MHz CTSD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, U3 ADF4159 FMCW PLL (RX LO chirp), U30 LT3045 ultra-low-noise LDO (R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, U31 LT3045 ultra-low-noise LDO (R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, U32 LT3045 ultra-low-noise LDO (R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, U33 LT3045 ultra-low-noise LDO (R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, U34 LT3045 ultra-low-noise LDO (R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, U35 LT3045 ultra-low-noise LDO (R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, U4 HMC733 VCO 10-20 GHz (LO), U40 ADP7159 LDO (ADC), U41 ADP7159 LDO (ADC), U42 ADP7159 LDO (ADC), U43 ADP7159 LDO (ADC), U44 ADP7159 LDO (ADC), U45 ADP7159 LDO (ADC), U5 HMC903 LO amp (+14 dBm), U50 ADAR1000 4-ch Ku beamformer (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, U51 ADAR1000 4-ch Ku beamformer (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, U60 Ku GaN-on-SiC PA 1 W (QGaN15,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, U61 Ku GaN-on-SiC PA 1 W (QGaN15,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, U62 Ku GaN-on-SiC PA 1 W (QGaN15,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, U63 Ku GaN-on-SiC PA 1 W (QGaN15,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, U64 Ku GaN-on-SiC PA 1 W (QGaN15,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, U65 Ku GaN-on-SiC PA 1 W (QGaN15,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, U8 HMC903 TX drive amp, U9 HMC7044 JESD204B clock + SYSR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, Y1 100 MHz OCXO, -165 dBc/Hz flo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

Commit message: Schematics, full-wave EM element optimisation, physical stack-ups
Schematics
- KiCad schematics for HG1-ANT/DSP/PWR generated by board/schematic/
  (33-symbol HG1 library, pins taken from the routed layout): ERC 0/0,
  schematic<->PCB parity clean; scripted "Update PCB from Schematic"
  links footprints, nets and values and stages unplaced parts.
- STM32G474 pin map corrected to the real LQFP-64 pin-out.

Full-wave EM of the radiating element (antenna/em, docs/06)
- EMerge FEM models: isolated element and infinite-array unit cell with
  a scan-matched Floquet port; local PARDISO and Modal (CPU, cuDSS GPU).
- Found and fixed: low slot/superstrate resonance of the analytic cut,
  60 deg azimuth scan blindness (element via-fence cavity), far-field
  dB scaling and E/H cut labelling.
- Differential evolution on Modal (792 solves, worst of 0/45/60 deg):
  driven 3.21 mm, parasitic 4.48 mm, slot 3.02 mm + 2.14 mm arms,
  stub 1.50 mm, 1.016 mm parasitic spacer. Active |S11| < -10 dB over
  0.52-0.70 GHz around 16 GHz at every scan to 60 az / 40 el.

Board / mechanical
- New element copper and 1,051 blind L1-L5 element-fence vias on ANT.
- Full physical stack-ups (hg1_params.STACKS) written into each
  .kicad_pcb; ANT is 2.716 mm (old 2.1 mm could not hold 10 layers).
- Enclosure, mass (1,059 g), KiCad and Blender renders regenerated.
  DRC 0 errors on all boards, parity clean.

Co-Authored-By: Claude Opus 5.5 <noreply@anthropic.com>
Parts:
- added C30: 10u, Capacitor_SMD:C_0805_2012Metric, F.Cu at (243.7, 38.0)
- added C31: 10u, Capacitor_SMD:C_0805_2012Metric, F.Cu at (251.2, 38.0)
- added C32: 10u, Capacitor_SMD:C_0805_2012Metric, F.Cu at (258.6, 38.0)
- added C33: 10u, Capacitor_SMD:C_0805_2012Metric, F.Cu at (266.1, 38.0)
- added C34: 10u, Capacitor_SMD:C_0805_2012Metric, F.Cu at (273.5, 38.0)
- added C35: 10u, Capacitor_SMD:C_0805_2012Metric, F.Cu at (281.0, 38.0)
- added C37: 47u, Capacitor_SMD:C_0805_2012Metric, F.Cu at (288.4, 38.0)
- added C40: 1u, Capacitor_SMD:C_0402_1005Metric, F.Cu at (295.1, 37.5)
- added C41: 1u, Capacitor_SMD:C_0402_1005Metric, F.Cu at (301.0, 37.5)
- added C42: 1u, Capacitor_SMD:C_0402_1005Metric, F.Cu at (306.8, 37.5)
- added C43: 1u, Capacitor_SMD:C_0402_1005Metric, F.Cu at (312.7, 37.5)
- added C44: 1u, Capacitor_SMD:C_0402_1005Metric, F.Cu at (318.6, 37.5)
- added C45: 1u, Capacitor_SMD:C_0402_1005Metric, F.Cu at (324.4, 37.5)
- added C50: 100n, Capacitor_SMD:C_0402_1005Metric, F.Cu at (330.3, 37.5)
- added C51: 100n, Capacitor_SMD:C_0402_1005Metric, F.Cu at (336.2, 37.5)
- added C52: 100n, Capacitor_SMD:C_0402_1005Metric, F.Cu at (342.0, 37.5)
- added C53: 100n, Capacitor_SMD:C_0402_1005Metric, F.Cu at (347.9, 37.5)
- added C54: 100n, Capacitor_SMD:C_0402_1005Metric, F.Cu at (353.8, 37.5)
- added C55: 100n, Capacitor_SMD:C_0402_1005Metric, F.Cu at (242.9, 43.5)
- added CLF1: 2.2n C0G loop filter, Capacitor_SMD:C_0402_1005Metric, F.Cu at (248.8, 43.5)
- added CLF3: 2.2n C0G loop filter, Capacitor_SMD:C_0402_1005Metric, F.Cu at (254.7, 43.5)
- added L1: 1u, Inductor_SMD:L_0805_2012Metric, F.Cu at (261.4, 43.9)
- added Q1: P-MOSFET -60 V drain switch, Package_SO:SOIC-8_3.9x4.9mm_P1.27mm, F.Cu at (270.9, 45.8)
- added Q2: 2N7002, Package_TO_SOT_SMD:SOT-23, F.Cu at (280.6, 44.7)
- added R10: 5.1k, Resistor_SMD:R_0402_1005Metric, F.Cu at (287.5, 43.5)
- added R100: 5.1k, Resistor_SMD:R_0402_1005Metric, F.Cu at (346.6, 43.5)
- added R30: 33.2k 0.1%, Resistor_SMD:R_0402_1005Metric, F.Cu at (293.4, 43.5)
- added R31: 33.2k 0.1%, Resistor_SMD:R_0402_1005Metric, F.Cu at (299.3, 43.5)
- added R32: 33.2k 0.1%, Resistor_SMD:R_0402_1005Metric, F.Cu at (305.2, 43.5)
- added R33: 33.2k 0.1%, Resistor_SMD:R_0402_1005Metric, F.Cu at (311.1, 43.5)
- added R34: 33.2k 0.1%, Resistor_SMD:R_0402_1005Metric, F.Cu at (317.0, 43.5)
- added R35: 33.2k 0.1%, Resistor_SMD:R_0402_1005Metric, F.Cu at (322.9, 43.5)
- added R36: 33.2k 0.1%, Resistor_SMD:R_0402_1005Metric, F.Cu at (328.8, 43.5)
- added R37: 20k, Resistor_SMD:R_0402_1005Metric, F.Cu at (334.8, 43.5)
- added R38: 80.6k, Resistor_SMD:R_0402_1005Metric, F.Cu at (340.7, 43.5)
- added RG1: 10k, Resistor_SMD:R_0402_1005Metric, F.Cu at (352.5, 43.5)
- added RG2: 10k, Resistor_SMD:R_0402_1005Metric, F.Cu at (243.0, 53.1)
- added RG3: 100k, Resistor_SMD:R_0402_1005Metric, F.Cu at (248.9, 53.1)
- added RP1: 10k 0.1%, Resistor_SMD:R_0402_1005Metric, F.Cu at (254.8, 53.1)
- added RP2: 10k 0.1%, Resistor_SMD:R_0402_1005Metric, F.Cu at (260.7, 53.1)
- added RP3: 10k 0.1%, Resistor_SMD:R_0402_1005Metric, F.Cu at (266.6, 53.1)
- added RP4: 10k 0.1%, Resistor_SMD:R_0402_1005Metric, F.Cu at (272.5, 53.1)
- added RP5: 10k 0.1%, Resistor_SMD:R_0402_1005Metric, F.Cu at (278.4, 53.1)
- added RP6: 10k 0.1%, Resistor_SMD:R_0402_1005Metric, F.Cu at (284.3, 53.1)
- added RS1: 10m 1% 0805, Resistor_SMD:R_0402_1005Metric, F.Cu at (290.2, 53.1)
- added RS2: 10m 1% 0805, Resistor_SMD:R_0402_1005Metric, F.Cu at (296.1, 53.1)
- added RS3: 10m 1% 0805, Resistor_SMD:R_0402_1005Metric, F.Cu at (302.1, 53.1)
- added RS4: 10m 1% 0805, Resistor_SMD:R_0402_1005Metric, F.Cu at (308.0, 53.1)
- added RS5: 10m 1% 0805, Resistor_SMD:R_0402_1005Metric, F.Cu at (313.9, 53.1)
- added RS6: 10m 1% 0805, Resistor_SMD:R_0402_1005Metric, F.Cu at (319.8, 53.1)
- added RT1: 10k B3435, Resistor_SMD:R_0402_1005Metric, F.Cu at (325.7, 53.1)
- added RT2: 10k B3435, Resistor_SMD:R_0402_1005Metric, F.Cu at (331.6, 53.1)
- added RT3: 10k B3435, Resistor_SMD:R_0402_1005Metric, F.Cu at (337.5, 53.1)
- added RT4: 10k B3435, Resistor_SMD:R_0402_1005Metric, F.Cu at (343.4, 53.1)
- added RT5: 10k B3435, Resistor_SMD:R_0402_1005Metric, F.Cu at (349.3, 53.1)
- added RT6: 10k B3435, Resistor_SMD:R_0402_1005Metric, F.Cu at (355.2, 53.1)
- added U36: LT3045 3.3 V (RF), Package_DFN_QFN:DFN-10-1EP_3x3mm_P0.5mm_EP1.65x2.38mm, F.Cu at (244.3, 59.4)
- added U37: TPS62913 1.0 V, Package_DFN_QFN:DFN-10-1EP_3x3mm_P0.5mm_EP1.65x2.38mm, F.Cu at (253.0, 59.4)
- added U39: ADS7138, Package_DFN_QFN:QFN-16-1EP_3x3mm_P0.5mm_EP1.7x1.7mm, F.Cu at (261.7, 59.7)
- added U70: INA186A3, Package_TO_SOT_SMD:SOT-363_SC-70-6, F.Cu at (269.5, 58.8)
- added U71: INA186A3, Package_TO_SOT_SMD:SOT-363_SC-70-6, F.Cu at (276.5, 58.8)
- added U72: INA186A3, Package_TO_SOT_SMD:SOT-363_SC-70-6, F.Cu at (283.4, 58.8)
- added U73: INA186A3, Package_TO_SOT_SMD:SOT-363_SC-70-6, F.Cu at (290.4, 58.8)
- added U74: INA186A3, Package_TO_SOT_SMD:SOT-363_SC-70-6, F.Cu at (297.3, 58.8)
- added U75: INA186A3, Package_TO_SOT_SMD:SOT-363_SC-70-6, F.Cu at (304.3, 58.8)
- AE1: value GNSS L1/L5 ceramic patch 18x18 (Taoglas CGGP.18 class) -> GNSS L1/L5 patch; footprint (none) -> HG1:GNSS_PATCH_18x18
- C1, C10, C11, C12, C2, C3, C4, C5, C6, C7, C8, C9: value 10u 50V X7R drain -> 10u 50V; footprint C_1210_3225Metric -> Capacitor_SMD:C_1210_3225Metric
- H1, H10, H2, H3, H4, H5, H6, H7, H8, H9: footprint MountingHole_2.7mm_M2.5_Pad_Via -> MountingHole:MountingHole_2.7mm_M2.5_Pad_Via
- J1: value Molex Micro-Fit 4p: +28V_PA, +5V, GND x2 -> Micro-Fit 4p power in; footprint Molex_Micro-Fit_3.0_43650-0400_1x04_P3.00mm_Horizontal -> Connector_Molex:Molex_Micro-Fit_3.0_43650-0400_1x04_P3.00mm_Horizontal
- J2, J3: value Samtec LSHM-150 JESD204B x12 lanes (10 mm stack) -> LSHM-150 JESD mezzanine; footprint Samtec_LSHM-150-xx.x-x-DV-N_2x50_P0.50mm_Vertical -> Connector_Samtec:Samtec_LSHM-150-xx.x-x-DV-N_2x50_P0.50mm_Vertical
- J4: value Samtec LSHM-120 SPI/sync/GNSS/RID/CAL -> LSHM-120 control mezzanine; footprint Samtec_LSHM-120-xx.x-x-DV-N_2x20_P0.50mm_Vertical -> Connector_Samtec:Samtec_LSHM-120-xx.x-x-DV-N_2x20_P0.50mm_Vertical
- U1: value ADF4159 FMCW PLL (TX chirp) -> ADF4159; footprint QFN-24-1EP_4x4mm_P0.5mm_EP2.6x2.6mm -> Package_DFN_QFN:QFN-24-1EP_4x4mm_P0.5mm_EP2.6x2.6mm
- U10, U11, U12, U13, U14, U15: value HRX-8 8-ch Ku SiGe RX RFIC (LNA+IQ mix+IF) -> HRX-8; footprint QFN-64-1EP_9x9mm_P0.5mm_EP3.8x3.8mm -> Package_DFN_QFN:QFN-64-1EP_9x9mm_P0.5mm_EP3.8x3.8mm
- U2: value HMC733 VCO 10-20 GHz (TX) -> HMC733LC4B; footprint QFN-24-1EP_4x4mm_P0.5mm_EP2.6x2.6mm -> Package_DFN_QFN:QFN-24-1EP_4x4mm_P0.5mm_EP2.6x2.6mm
- U20, U21, U22, U23, U24, U25: value AD9083BBCZ 16-ch 125 MHz CTSD ADC -> AD9083BBCZ; footprint BGA-121_9.0x9.0mm_Layout11x11_P0.8mm_Ball0.4mm_Pad0.35mm_NSMD -> Package_BGA:BGA-121_9.0x9.0mm_Layout11x11_P0.8mm_Ball0.4mm_Pad0.35mm_NSMD
- U3: value ADF4159 FMCW PLL (RX LO chirp) -> ADF4159; footprint QFN-24-1EP_4x4mm_P0.5mm_EP2.6x2.6mm -> Package_DFN_QFN:QFN-24-1EP_4x4mm_P0.5mm_EP2.6x2.6mm
- U30, U31, U32, U33, U34, U35: value LT3045 ultra-low-noise LDO (RFIC) -> LT3045 3.3 V; footprint DFN-10-1EP_3x3mm_P0.5mm_EP1.65x2.38mm -> Package_DFN_QFN:DFN-10-1EP_3x3mm_P0.5mm_EP1.65x2.38mm
- U4: value HMC733 VCO 10-20 GHz (LO) -> HMC733LC4B; footprint QFN-24-1EP_4x4mm_P0.5mm_EP2.6x2.6mm -> Package_DFN_QFN:QFN-24-1EP_4x4mm_P0.5mm_EP2.6x2.6mm
- U40, U41, U42, U43, U44, U45: value ADP7159 LDO (ADC) -> ADP7159 1.8 V; footprint DFN-10-1EP_3x3mm_P0.5mm_EP1.65x2.38mm -> Package_DFN_QFN:DFN-10-1EP_3x3mm_P0.5mm_EP1.65x2.38mm
- U5: value HMC903 LO amp (+14 dBm) -> HMC903LP3E; footprint QFN-16-1EP_3x3mm_P0.5mm_EP1.7x1.7mm -> Package_DFN_QFN:QFN-16-1EP_3x3mm_P0.5mm_EP1.7x1.7mm
- U50, U51: value ADAR1000 4-ch Ku beamformer (DDMA phase code / spotlight) -> ADAR1000; footprint QFN-48-1EP_7x7mm_P0.5mm_EP5.6x5.6mm_ThermalVias -> Package_DFN_QFN:QFN-48-1EP_7x7mm_P0.5mm_EP5.6x5.6mm_ThermalVias
- U60, U61, U62, U63, U64, U65: value Ku GaN-on-SiC PA 1 W (QGaN15, 28 V) -> GaN PA 1 W; footprint QFN-24-1EP_4x4mm_P0.5mm_EP2.65x2.65mm_ThermalVias -> Package_DFN_QFN:QFN-24-1EP_4x4mm_P0.5mm_EP2.65x2.65mm_ThermalVias
- U8: value HMC903 TX drive amp -> HMC903LP3E; footprint QFN-16-1EP_3x3mm_P0.5mm_EP1.7x1.7mm -> Package_DFN_QFN:QFN-16-1EP_3x3mm_P0.5mm_EP1.7x1.7mm
- U9: value HMC7044 JESD204B clock + SYSREF (14 out) -> HMC7044; footprint QFN-64-1EP_9x9mm_P0.5mm_EP3.8x3.8mm -> Package_DFN_QFN:QFN-64-1EP_9x9mm_P0.5mm_EP3.8x3.8mm
- Y1: value 100 MHz OCXO, -165 dBc/Hz floor -> 100 MHz OCXO; footprint Oscillator_SMD_Diodes_FN-4Pin_7.0x5.0mm -> Oscillator:Oscillator_SMD_Diodes_FN-4Pin_7.0x5.0mm
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Connections:
- C1 pad 1: (no net) -> PA_D1
- C1 pad 2: (no net) -> GND
- C10 pad 1: (no net) -> PA_D5
- C10 pad 2: (no net) -> GND
- C11 pad 1: (no net) -> PA_D6
- C11 pad 2: (no net) -> GND
- C12 pad 1: (no net) -> PA_D6
- C12 pad 2: (no net) -> GND
- C2 pad 1: (no net) -> PA_D1
- C2 pad 2: (no net) -> GND
- C3 pad 1: (no net) -> PA_D2
- C3 pad 2: (no net) -> GND
- C4 pad 1: (no net) -> PA_D2
- C4 pad 2: (no net) -> GND
- C5 pad 1: (no net) -> PA_D3
- C5 pad 2: (no net) -> GND
- C6 pad 1: (no net) -> PA_D3
- C6 pad 2: (no net) -> GND
- C7 pad 1: (no net) -> PA_D4
- C7 pad 2: (no net) -> GND
- C8 pad 1: (no net) -> PA_D4
- C8 pad 2: (no net) -> GND
- C9 pad 1: (no net) -> PA_D5
- C9 pad 2: (no net) -> GND
- J1 pad 1: (no net) -> +28V_PA
- J1 pad 2: (no net) -> +5V
- J1 pad 3: (no net) -> GND
- J1 pad 4: (no net) -> GND
- J2 pad 1: (no net) -> GND
- J2 pad 10: (no net) -> GND
- J2 pad 11: (no net) -> GND
- J2 pad 12: (no net) -> GND
- J2 pad 13: (no net) -> GND
- J2 pad 14: (no net) -> GND
- J2 pad 15: (no net) -> GND
- J2 pad 16: (no net) -> GND
- J2 pad 17: (no net) -> GND
- J2 pad 18: (no net) -> GND
- J2 pad 19: (no net) -> GND
- J2 pad 21: (no net) -> GND
- J2 pad 22: (no net) -> GND
- J2 pad 23: (no net) -> GND
- J2 pad 25: (no net) -> GND
- J2 pad 27: (no net) -> GND
- J2 pad 28: (no net) -> GND
- J2 pad 29: (no net) -> GND
- J2 pad 3: (no net) -> CAL_PROBE
- J2 pad 31: (no net) -> GND
- J2 pad 32: (no net) -> GND
- J2 pad 33: (no net) -> GND
- J2 pad 34: (no net) -> GND
- J2 pad 35: (no net) -> GND
- J2 pad 36: (no net) -> GND
- J2 pad 37: (no net) -> GND
- J2 pad 38: (no net) -> GND
- J2 pad 39: (no net) -> GND
- J2 pad 40: (no net) -> GND
- J2 pad 41: (no net) -> GND
- J2 pad 42: (no net) -> GND
- J2 pad 43: (no net) -> GND
- J2 pad 44: (no net) -> GND
- J2 pad 45: (no net) -> GND
- J2 pad 46: (no net) -> GND
- J2 pad 47: (no net) -> GND
- J2 pad 48: (no net) -> GND
- J2 pad 49: (no net) -> GND
- J2 pad 5: (no net) -> CAL_PROBE
- J2 pad 50: (no net) -> GND
- J2 pad 51: (no net) -> GND
- J2 pad 52: (no net) -> GND
- J2 pad 53: (no net) -> GND
- J2 pad 54: (no net) -> GND
- J2 pad 55: (no net) -> GND
- J2 pad 56: (no net) -> GND
- J2 pad 57: (no net) -> GND
- J2 pad 58: (no net) -> GND
- J2 pad 59: (no net) -> GND
- J2 pad 60: (no net) -> GND
- J2 pad 61: (no net) -> GND
- J2 pad 62: (no net) -> GND
- J2 pad 63: (no net) -> GND
- J2 pad 64: (no net) -> GND
- J2 pad 65: (no net) -> GND
- J2 pad 66: (no net) -> GND
- J2 pad 67: (no net) -> GND
- J2 pad 68: (no net) -> GND
- J2 pad 69: (no net) -> GND
- J2 pad 7: (no net) -> CAL_PROBE
- J2 pad 70: (no net) -> GND
- J2 pad 71: (no net) -> GND
- J2 pad 72: (no net) -> GND
- J2 pad 73: (no net) -> GND
- J2 pad 74: (no net) -> GND
- J2 pad 75: (no net) -> GND
- J2 pad 76: (no net) -> GND
- J2 pad 77: (no net) -> GND
- J2 pad 78: (no net) -> GND
- J2 pad 79: (no net) -> GND
- J2 pad 80: (no net) -> GND
- J2 pad 81: (no net) -> GND
- J2 pad 82: (no net) -> GND
- J2 pad 83: (no net) -> GND
- J2 pad 84: (no net) -> GND
- J2 pad 85: (no net) -> GND
- J2 pad 86: (no net) -> GND
- J2 pad 87: (no net) -> GND
- J2 pad 88: (no net) -> GND
- J2 pad 89: (no net) -> GND
- J2 pad 9: (no net) -> CAL_PROBE
- J2 pad 90: (no net) -> GND
- J2 pad 91: (no net) -> GND
- J2 pad 93: (no net) -> GND
- J2 pad 94: (no net) -> GND
- J2 pad 95: (no net) -> GND
- J2 pad 97: (no net) -> GND
- J2 pad 99: (no net) -> GND
- J3 pad 1: (no net) -> GND
- J3 pad 100: JESD4_L3 -> JESD4_L0
- J3 pad 11: (no net) -> ID_PA2
- J3 pad 12: (no net) -> GND
- J3 pad 13: (no net) -> GND
- J3 pad 15: (no net) -> ID_PA3
- J3 pad 16: (no net) -> GND
- J3 pad 17: (no net) -> ID_PA4
- J3 pad 18: (no net) -> GND
- J3 pad 19: (no net) -> ID_PA5
- J3 pad 2: (no net) -> GND
- J3 pad 20: (no net) -> GND
- J3 pad 21: (no net) -> ID_PA6
- J3 pad 22: (no net) -> GND
- J3 pad 23: (no net) -> ID_PA1
- J3 pad 24: (no net) -> GND
- J3 pad 25: (no net) -> ID_PA2
- J3 pad 26: (no net) -> GND
- J3 pad 27: (no net) -> ID_PA3
- J3 pad 28: (no net) -> GND
- J3 pad 29: (no net) -> ID_PA4
- J3 pad 3: (no net) -> GND
- J3 pad 30: (no net) -> GND
- J3 pad 31: (no net) -> ID_PA5
- J3 pad 32: (no net) -> GND
- J3 pad 33: (no net) -> ID_PA6
- J3 pad 34: (no net) -> GND
- J3 pad 35: (no net) -> ID_PA1
- J3 pad 36: (no net) -> GND
- J3 pad 37: (no net) -> ID_PA2
- J3 pad 38: (no net) -> GND
- J3 pad 39: (no net) -> ID_PA3
- J3 pad 40: (no net) -> GND
- J3 pad 41: (no net) -> ID_PA4
- J3 pad 42: (no net) -> GND
- J3 pad 43: (no net) -> ID_PA5
- J3 pad 44: (no net) -> GND
- J3 pad 45: (no net) -> ID_PA6
- J3 pad 46: (no net) -> GND
- J3 pad 47: (no net) -> ID_PA1
- J3 pad 48: (no net) -> GND
- J3 pad 49: (no net) -> ID_PA2
- J3 pad 5: (no net) -> ID_PA1
- J3 pad 50: (no net) -> GND
- J3 pad 51: (no net) -> ID_PA3
- J3 pad 52: (no net) -> GND
- J3 pad 53: (no net) -> ID_PA4
- J3 pad 54: (no net) -> GND
- J3 pad 55: (no net) -> ID_PA5
- J3 pad 56: (no net) -> GND
- J3 pad 57: (no net) -> ID_PA6
- J3 pad 58: (no net) -> GND
- J3 pad 59: (no net) -> GND
- J3 pad 6: (no net) -> GND
- J3 pad 60: (no net) -> GND
- J3 pad 61: (no net) -> GND
- J3 pad 62: (no net) -> GND
- J3 pad 63: (no net) -> GND
- J3 pad 64: (no net) -> GND
- J3 pad 65: (no net) -> GND
- J3 pad 66: (no net) -> GND
- J3 pad 67: (no net) -> GND
- J3 pad 68: (no net) -> GND
- J3 pad 69: (no net) -> GND
- J3 pad 7: (no net) -> GND
- J3 pad 70: (no net) -> GND
- J3 pad 71: (no net) -> GND
- J3 pad 72: (no net) -> GND
- J3 pad 73: (no net) -> GND
- J3 pad 74: (no net) -> GND
- J3 pad 75: (no net) -> GND
- J3 pad 77: (no net) -> GND
- J3 pad 78: (no net) -> GND
- J3 pad 79: (no net) -> GND
- J3 pad 81: (no net) -> GND
- J3 pad 83: (no net) -> GND
- J3 pad 84: (no net) -> GND
- J3 pad 85: (no net) -> GND
- J3 pad 87: (no net) -> GND
- J3 pad 88: (no net) -> GND
- J3 pad 89: (no net) -> GND
- J3 pad 9: (no net) -> GND
- J3 pad 90: (no net) -> GND
- J3 pad 91: (no net) -> GND
- J3 pad 92: (no net) -> GND
- J3 pad 93: (no net) -> GND
- J3 pad 94: JESD4_L0 -> JESD4_L3
- J3 pad 95: (no net) -> GND
- J3 pad 96: JESD4_L1 -> JESD4_L2
- J3 pad 97: (no net) -> GND
- J3 pad 98: JESD4_L2 -> JESD4_L1
- J3 pad 99: (no net) -> GND
- J4 pad 1: (no net) -> SPI_SCLK
- J4 pad 10: (no net) -> CS_ADC0
- J4 pad 11: (no net) -> CS_ADC1
- J4 pad 12: (no net) -> CS_ADC2
- J4 pad 13: (no net) -> CS_ADC3
- J4 pad 14: (no net) -> CS_ADC4
- J4 pad 15: (no net) -> CS_ADC5
- J4 pad 16: (no net) -> CS_PLL_TX
- J4 pad 17: (no net) -> CS_PLL_LO
- J4 pad 18: (no net) -> CS_CLK
- J4 pad 19: (no net) -> CHIRP_TRIG
- J4 pad 2: (no net) -> GND
- J4 pad 20: (no net) -> JESD_SYNC
- J4 pad 21: (no net) -> PLL_LD_TX
- J4 pad 22: (no net) -> PLL_LD_LO
- J4 pad 23: (no net) -> FPGA_REFCLK
- J4 pad 24: (no net) -> FPGA_SYSREF
- J4 pad 25: (no net) -> MCU_SPI_SCK
- J4 pad 26: (no net) -> MCU_SPI_MOSI
- J4 pad 27: (no net) -> MCU_SPI_MISO
- J4 pad 28: (no net) -> CS_BF0
- J4 pad 29: (no net) -> CS_BF1
- J4 pad 3: (no net) -> SPI_MOSI
- J4 pad 30: (no net) -> TX_MUTE_N
- J4 pad 31: (no net) -> TX_LOAD
- J4 pad 32: (no net) -> EN_DRAIN_SW
- J4 pad 33: (no net) -> I2C3_SCL
- J4 pad 34: (no net) -> I2C3_SDA
- J4 pad 35: (no net) -> GNSS_RF
- J4 pad 36: (no net) -> RID_RF
- J4 pad 37: (no net) -> -5V_BIAS
- J4 pad 38: (no net) -> RF_RESET_N
- J4 pad 39: (no net) -> GND
- J4 pad 4: (no net) -> CS_RFIC0
- J4 pad 40: (no net) -> GND
- J4 pad 5: (no net) -> CS_RFIC1
- J4 pad 6: (no net) -> CS_RFIC2
- J4 pad 7: (no net) -> CS_RFIC3
- J4 pad 8: (no net) -> CS_RFIC4
- J4 pad 9: (no net) -> CS_RFIC5
- U1 pad 12: (no net) -> CHIRP_TRIG
- U1 pad 13: (no net) -> SPI_SCLK
- U1 pad 14: (no net) -> SPI_MOSI
- U1 pad 15: (no net) -> CS_PLL_TX
- U1 pad 16: (no net) -> +3V3_RF
- U1 pad 18: (no net) -> PLL_LD_TX
- U1 pad 20: (no net) -> RSET_TX
- U1 pad 5: (no net) -> +3V3_RF
- U1 pad 6: (no net) -> +3V3_RF
- U1 pad 7: (no net) -> +3V3_RF
- U1 pad 8: (no net) -> +3V3_RF
- U1 pad 9: (no net) -> TX_VCO_DIV
- U10 pad 1: (no net) -> GND
- U10 pad 10: (no net) -> GND
- U10 pad 12: (no net) -> GND
- U10 pad 13: (no net) -> VCC_RX1
- U10 pad 14: (no net) -> GND
- U10 pad 16: (no net) -> GND
- U10 pad 17: (no net) -> SPI_SCLK
- U10 pad 18: (no net) -> SPI_MOSI
- U10 pad 19: (no net) -> CS_RFIC0
- U10 pad 20: (no net) -> RF_RESET_N
- U10 pad 21: (no net) -> GND
- U10 pad 22: (no net) -> unconnected-(U10-TEMP-Pad22)
- U10 pad 23: (no net) -> GND
- U10 pad 25: (no net) -> GND
- U10 pad 26: (no net) -> VCC_RX1
- U10 pad 27: (no net) -> VCM1
- U10 pad 3: (no net) -> GND
- U10 pad 30: (no net) -> GND
- U10 pad 31: (no net) -> GND
- U10 pad 32: (no net) -> GND
- U10 pad 33: (no net) -> GND
- U10 pad 35: (no net) -> GND
- U10 pad 36: (no net) -> VCC_RX1
- U10 pad 37: (no net) -> GND
- U10 pad 39: (no net) -> GND
- U10 pad 4: (no net) -> VCC_RX1
- U10 pad 40: (no net) -> VCC_RX1
- U10 pad 41: (no net) -> VCC_RX1
- U10 pad 42: (no net) -> GND
- U10 pad 44: (no net) -> GND
- U10 pad 45: (no net) -> VCC_RX1
- U10 pad 46: (no net) -> GND
- U10 pad 48: (no net) -> GND
- U10 pad 5: (no net) -> GND
- U10 pad 7: (no net) -> GND
- U10 pad 8: (no net) -> VCC_RX1
- U10 pad 9: (no net) -> VCC_RX1
- U11 pad 1: (no net) -> GND
- U11 pad 10: (no net) -> GND
- U11 pad 12: (no net) -> GND
- U11 pad 13: (no net) -> VCC_RX2
- U11 pad 14: (no net) -> GND
- U11 pad 16: (no net) -> GND
- U11 pad 17: (no net) -> SPI_SCLK
- U11 pad 18: (no net) -> SPI_MOSI
- U11 pad 19: (no net) -> CS_RFIC1
- U11 pad 20: (no net) -> RF_RESET_N
- U11 pad 21: (no net) -> GND
- U11 pad 22: (no net) -> unconnected-(U11-TEMP-Pad22)
- U11 pad 23: (no net) -> GND
- U11 pad 25: (no net) -> GND
- U11 pad 26: (no net) -> VCC_RX2
- U11 pad 27: (no net) -> VCM2
- U11 pad 3: (no net) -> GND
- U11 pad 30: (no net) -> GND
- U11 pad 31: (no net) -> GND
- U11 pad 32: (no net) -> GND
- U11 pad 33: (no net) -> GND
- U11 pad 35: (no net) -> GND
- U11 pad 36: (no net) -> VCC_RX2
- U11 pad 37: (no net) -> GND
- U11 pad 39: (no net) -> GND
- U11 pad 4: (no net) -> VCC_RX2
- U11 pad 40: (no net) -> VCC_RX2
- U11 pad 41: (no net) -> VCC_RX2
- U11 pad 42: (no net) -> GND
- U11 pad 44: (no net) -> GND
- U11 pad 45: (no net) -> VCC_RX2
- U11 pad 46: (no net) -> GND
- U11 pad 48: (no net) -> GND
- U11 pad 5: (no net) -> GND
- U11 pad 7: (no net) -> GND
- U11 pad 8: (no net) -> VCC_RX2
- U11 pad 9: (no net) -> VCC_RX2
- U12 pad 1: (no net) -> GND
- U12 pad 10: (no net) -> GND
- U12 pad 12: (no net) -> GND
- U12 pad 13: (no net) -> VCC_RX3
- U12 pad 14: (no net) -> GND
- U12 pad 16: (no net) -> GND
- U12 pad 17: (no net) -> SPI_SCLK
- U12 pad 18: (no net) -> SPI_MOSI
- U12 pad 19: (no net) -> CS_RFIC2
- U12 pad 20: (no net) -> RF_RESET_N
- U12 pad 21: (no net) -> GND
- U12 pad 22: (no net) -> unconnected-(U12-TEMP-Pad22)
- U12 pad 23: (no net) -> GND
- U12 pad 25: (no net) -> GND
- U12 pad 26: (no net) -> VCC_RX3
- U12 pad 27: (no net) -> VCM3
- U12 pad 3: (no net) -> GND
- U12 pad 30: (no net) -> GND
- U12 pad 31: (no net) -> GND
- U12 pad 32: (no net) -> GND
- U12 pad 33: (no net) -> GND
- U12 pad 35: (no net) -> GND
- U12 pad 36: (no net) -> VCC_RX3
- U12 pad 37: (no net) -> GND
- U12 pad 39: (no net) -> GND
- U12 pad 4: (no net) -> VCC_RX3
- U12 pad 40: (no net) -> VCC_RX3
- U12 pad 41: (no net) -> VCC_RX3
- U12 pad 42: (no net) -> GND
- U12 pad 44: (no net) -> GND
- U12 pad 45: (no net) -> VCC_RX3
- U12 pad 46: (no net) -> GND
- U12 pad 48: (no net) -> GND
- U12 pad 5: (no net) -> GND
- U12 pad 7: (no net) -> GND
- U12 pad 8: (no net) -> VCC_RX3
- U12 pad 9: (no net) -> VCC_RX3
- U13 pad 1: (no net) -> GND
- U13 pad 10: (no net) -> GND
- U13 pad 12: (no net) -> GND
- U13 pad 13: (no net) -> VCC_RX4
- U13 pad 14: (no net) -> GND
- U13 pad 16: (no net) -> GND
- U13 pad 17: (no net) -> SPI_SCLK
- U13 pad 18: (no net) -> SPI_MOSI
- U13 pad 19: (no net) -> CS_RFIC3
- U13 pad 20: (no net) -> RF_RESET_N
- U13 pad 21: (no net) -> GND
- U13 pad 22: (no net) -> unconnected-(U13-TEMP-Pad22)
- U13 pad 23: (no net) -> GND
- U13 pad 25: (no net) -> GND
- U13 pad 26: (no net) -> VCC_RX4
- U13 pad 27: (no net) -> VCM4
- U13 pad 3: (no net) -> GND
- U13 pad 30: (no net) -> GND
- U13 pad 31: (no net) -> GND
- U13 pad 32: (no net) -> GND
- U13 pad 33: (no net) -> GND
- U13 pad 35: (no net) -> GND
- U13 pad 36: (no net) -> VCC_RX4
- U13 pad 37: (no net) -> GND
- U13 pad 39: (no net) -> GND
- U13 pad 4: (no net) -> VCC_RX4
- U13 pad 40: (no net) -> VCC_RX4
- U13 pad 41: (no net) -> VCC_RX4
- U13 pad 42: (no net) -> GND
- U13 pad 44: (no net) -> GND
- U13 pad 45: (no net) -> VCC_RX4
- U13 pad 46: (no net) -> GND
- U13 pad 48: (no net) -> GND
- U13 pad 5: (no net) -> GND
- U13 pad 7: (no net) -> GND
- U13 pad 8: (no net) -> VCC_RX4
- U13 pad 9: (no net) -> VCC_RX4
- U14 pad 1: (no net) -> GND
- U14 pad 10: (no net) -> GND
- U14 pad 12: (no net) -> GND
- U14 pad 13: (no net) -> VCC_RX5
- U14 pad 14: (no net) -> GND
- U14 pad 16: (no net) -> GND
- U14 pad 17: (no net) -> SPI_SCLK
- U14 pad 18: (no net) -> SPI_MOSI
- U14 pad 19: (no net) -> CS_RFIC4
- U14 pad 20: (no net) -> RF_RESET_N
- U14 pad 21: (no net) -> GND
- U14 pad 22: (no net) -> unconnected-(U14-TEMP-Pad22)
- U14 pad 23: (no net) -> GND
- U14 pad 25: (no net) -> GND
- U14 pad 26: (no net) -> VCC_RX5
- U14 pad 27: (no net) -> VCM5
- U14 pad 3: (no net) -> GND
- U14 pad 30: (no net) -> GND
- U14 pad 31: (no net) -> GND
- U14 pad 32: (no net) -> GND
- U14 pad 33: (no net) -> GND
- U14 pad 35: (no net) -> GND
- U14 pad 36: (no net) -> VCC_RX5
- U14 pad 37: (no net) -> GND
- U14 pad 39: (no net) -> GND
- U14 pad 4: (no net) -> VCC_RX5
- U14 pad 40: (no net) -> VCC_RX5
- U14 pad 41: (no net) -> VCC_RX5
- U14 pad 42: (no net) -> GND
- U14 pad 44: (no net) -> GND
- U14 pad 45: (no net) -> VCC_RX5
- U14 pad 46: (no net) -> GND
- U14 pad 48: (no net) -> GND
- U14 pad 5: (no net) -> GND
- U14 pad 7: (no net) -> GND
- U14 pad 8: (no net) -> VCC_RX5
- U14 pad 9: (no net) -> VCC_RX5
- U15 pad 1: (no net) -> GND
- U15 pad 10: (no net) -> GND
- U15 pad 12: (no net) -> GND
- U15 pad 13: (no net) -> VCC_RX6
- U15 pad 14: (no net) -> GND
- U15 pad 16: (no net) -> GND
- U15 pad 17: (no net) -> SPI_SCLK
- U15 pad 18: (no net) -> SPI_MOSI
- U15 pad 19: (no net) -> CS_RFIC5
- U15 pad 20: (no net) -> RF_RESET_N
- U15 pad 21: (no net) -> GND
- U15 pad 22: (no net) -> unconnected-(U15-TEMP-Pad22)
- U15 pad 23: (no net) -> GND
- U15 pad 25: (no net) -> GND
- U15 pad 26: (no net) -> VCC_RX6
- U15 pad 27: (no net) -> VCM6
- U15 pad 3: (no net) -> GND
- U15 pad 30: (no net) -> GND
- U15 pad 31: (no net) -> GND
- U15 pad 32: (no net) -> GND
- U15 pad 33: (no net) -> GND
- U15 pad 35: (no net) -> GND
- U15 pad 36: (no net) -> VCC_RX6
- U15 pad 37: (no net) -> GND
- U15 pad 39: (no net) -> GND
- U15 pad 4: (no net) -> VCC_RX6
- U15 pad 40: (no net) -> VCC_RX6
- U15 pad 41: (no net) -> VCC_RX6
- U15 pad 42: (no net) -> GND
- U15 pad 44: (no net) -> GND
- U15 pad 45: (no net) -> VCC_RX6
- U15 pad 46: (no net) -> GND
- U15 pad 48: (no net) -> GND
- U15 pad 5: (no net) -> GND
- U15 pad 7: (no net) -> GND
- U15 pad 8: (no net) -> VCC_RX6
- U15 pad 9: (no net) -> VCC_RX6
- U2 pad 21: (no net) -> TX_VCO_DIV
- U2 pad 3: (no net) -> +5V
- U2 pad 4: (no net) -> +5V
- U20 pad A10: (no net) -> ADC_SYSREF1
- U20 pad A11: (no net) -> unconnected-(U20-SYSREF--PadA11)
- U20 pad A2: (no net) -> ADC_CLK1
- U20 pad A3: (no net) -> unconnected-(U20-CLK--PadA3)
- U20 pad B1: (no net) -> JESD_SYNC
- U20 pad C1: (no net) -> SPI_SCLK
- U20 pad C2: (no net) -> SPI_MOSI
- U20 pad C3: (no net) -> CS_ADC0
- U20 pad C4: (no net) -> GND
- U20 pad D1: (no net) -> VCM1
- U20 pad E1: (no net) -> GND
- U20 pad E2: (no net) -> GND
- U20 pad E5: (no net) -> +1V0_ADC
- U20 pad E6: (no net) -> +1V0_ADC
- U20 pad E7: (no net) -> +1V0_ADC
- U20 pad F2: (no net) -> GND
- U20 pad F5: (no net) -> AVDD1P8_1
- U20 pad F6: (no net) -> AVDD1P8_1
- U20 pad F7: (no net) -> AVDD1P8_1
- U20 pad G5: (no net) -> GND
- U20 pad G6: (no net) -> GND
- U20 pad G7: (no net) -> GND
- U20 pad H5: (no net) -> GND
- U20 pad H6: (no net) -> GND
- U21 pad A10: (no net) -> ADC_SYSREF2
- U21 pad A11: (no net) -> unconnected-(U21-SYSREF--PadA11)
- U21 pad A2: (no net) -> ADC_CLK2
- U21 pad A3: (no net) -> unconnected-(U21-CLK--PadA3)
- U21 pad B1: (no net) -> JESD_SYNC
- U21 pad C1: (no net) -> SPI_SCLK
- U21 pad C2: (no net) -> SPI_MOSI
- U21 pad C3: (no net) -> CS_ADC1
- U21 pad C4: (no net) -> GND
- U21 pad D1: (no net) -> VCM2
- U21 pad E1: (no net) -> GND
- U21 pad E2: (no net) -> GND
- U21 pad E5: (no net) -> +1V0_ADC
- U21 pad E6: (no net) -> +1V0_ADC
- U21 pad E7: (no net) -> +1V0_ADC
- U21 pad F2: (no net) -> GND
- U21 pad F5: (no net) -> AVDD1P8_2
- U21 pad F6: (no net) -> AVDD1P8_2
- U21 pad F7: (no net) -> AVDD1P8_2
- U21 pad G5: (no net) -> GND
- U21 pad G6: (no net) -> GND
- U21 pad G7: (no net) -> GND
- U21 pad H5: (no net) -> GND
- U21 pad H6: (no net) -> GND
- U22 pad A10: (no net) -> ADC_SYSREF3
- U22 pad A11: (no net) -> unconnected-(U22-SYSREF--PadA11)
- U22 pad A2: (no net) -> ADC_CLK3
- U22 pad A3: (no net) -> unconnected-(U22-CLK--PadA3)
- U22 pad B1: (no net) -> JESD_SYNC
- U22 pad C1: (no net) -> SPI_SCLK
- U22 pad C2: (no net) -> SPI_MOSI
- U22 pad C3: (no net) -> CS_ADC2
- U22 pad C4: (no net) -> GND
- U22 pad D1: (no net) -> VCM3
- U22 pad E1: (no net) -> GND
- U22 pad E2: (no net) -> GND
- U22 pad E5: (no net) -> +1V0_ADC
- U22 pad E6: (no net) -> +1V0_ADC
- U22 pad E7: (no net) -> +1V0_ADC
- U22 pad F2: (no net) -> GND
- U22 pad F5: (no net) -> AVDD1P8_3
- U22 pad F6: (no net) -> AVDD1P8_3
- U22 pad F7: (no net) -> AVDD1P8_3
- U22 pad G5: (no net) -> GND
- U22 pad G6: (no net) -> GND
- U22 pad G7: (no net) -> GND
- U22 pad H5: (no net) -> GND
- U22 pad H6: (no net) -> GND
- U23 pad A10: (no net) -> ADC_SYSREF4
- U23 pad A11: (no net) -> unconnected-(U23-SYSREF--PadA11)
- U23 pad A2: (no net) -> ADC_CLK4
- U23 pad A3: (no net) -> unconnected-(U23-CLK--PadA3)
- U23 pad A5: JESD4_L0 -> JESD4_L3
- U23 pad A6: JESD4_L1 -> JESD4_L2
- U23 pad A7: JESD4_L2 -> JESD4_L1
- U23 pad A8: JESD4_L3 -> JESD4_L0
- U23 pad B1: (no net) -> JESD_SYNC
- U23 pad C1: (no net) -> SPI_SCLK
- U23 pad C2: (no net) -> SPI_MOSI
- U23 pad C3: (no net) -> CS_ADC3
- U23 pad C4: (no net) -> GND
- U23 pad D1: (no net) -> VCM4
- U23 pad E1: (no net) -> GND
- U23 pad E2: (no net) -> GND
- U23 pad E5: (no net) -> +1V0_ADC
- U23 pad E6: (no net) -> +1V0_ADC
- U23 pad E7: (no net) -> +1V0_ADC
- U23 pad F2: (no net) -> GND
- U23 pad F5: (no net) -> AVDD1P8_4
- U23 pad F6: (no net) -> AVDD1P8_4
- U23 pad F7: (no net) -> AVDD1P8_4
- U23 pad G5: (no net) -> GND
- U23 pad G6: (no net) -> GND
- U23 pad G7: (no net) -> GND
- U23 pad H5: (no net) -> GND
- U23 pad H6: (no net) -> GND
- U24 pad A10: (no net) -> ADC_SYSREF5
- U24 pad A11: (no net) -> unconnected-(U24-SYSREF--PadA11)
- U24 pad A2: (no net) -> ADC_CLK5
- U24 pad A3: (no net) -> unconnected-(U24-CLK--PadA3)
- U24 pad B1: (no net) -> JESD_SYNC
- U24 pad C1: (no net) -> SPI_SCLK
- U24 pad C2: (no net) -> SPI_MOSI
- U24 pad C3: (no net) -> CS_ADC4
- U24 pad C4: (no net) -> GND
- U24 pad D1: (no net) -> VCM5
- U24 pad E1: (no net) -> GND
- U24 pad E2: (no net) -> GND
- U24 pad E5: (no net) -> +1V0_ADC
- U24 pad E6: (no net) -> +1V0_ADC
- U24 pad E7: (no net) -> +1V0_ADC
- U24 pad F2: (no net) -> GND
- U24 pad F5: (no net) -> AVDD1P8_5
- U24 pad F6: (no net) -> AVDD1P8_5
- U24 pad F7: (no net) -> AVDD1P8_5
- U24 pad G5: (no net) -> GND
- U24 pad G6: (no net) -> GND
- U24 pad G7: (no net) -> GND
- U24 pad H5: (no net) -> GND
- U24 pad H6: (no net) -> GND
- U25 pad A10: (no net) -> ADC_SYSREF6
- U25 pad A11: (no net) -> unconnected-(U25-SYSREF--PadA11)
- U25 pad A2: (no net) -> ADC_CLK6
- U25 pad A3: (no net) -> unconnected-(U25-CLK--PadA3)
- U25 pad B1: (no net) -> JESD_SYNC
- U25 pad C1: (no net) -> SPI_SCLK
- U25 pad C2: (no net) -> SPI_MOSI
- U25 pad C3: (no net) -> CS_ADC5
- U25 pad C4: (no net) -> GND
- U25 pad D1: (no net) -> VCM6
- U25 pad E1: (no net) -> GND
- U25 pad E2: (no net) -> GND
- U25 pad E5: (no net) -> +1V0_ADC
- U25 pad E6: (no net) -> +1V0_ADC
- U25 pad E7: (no net) -> +1V0_ADC
- U25 pad F2: (no net) -> GND
- U25 pad F5: (no net) -> AVDD1P8_6
- U25 pad F6: (no net) -> AVDD1P8_6
- U25 pad F7: (no net) -> AVDD1P8_6
- U25 pad G5: (no net) -> GND
- U25 pad G6: (no net) -> GND
- U25 pad G7: (no net) -> GND
- U25 pad H5: (no net) -> GND
- U25 pad H6: (no net) -> GND
- U3 pad 12: (no net) -> CHIRP_TRIG
- U3 pad 13: (no net) -> SPI_SCLK
- U3 pad 14: (no net) -> SPI_MOSI
- U3 pad 15: (no net) -> CS_PLL_LO
- U3 pad 16: (no net) -> +3V3_RF
- U3 pad 18: (no net) -> PLL_LD_LO
- U3 pad 20: (no net) -> RSET_LO
- U3 pad 5: (no net) -> +3V3_RF
- U3 pad 6: (no net) -> +3V3_RF
- U3 pad 7: (no net) -> +3V3_RF
- U3 pad 8: (no net) -> +3V3_RF
- U3 pad 9: (no net) -> LO_VCO_DIV
- U30 pad 1: (no net) -> +5V
- U30 pad 10: (no net) -> VCC_RX1
- U30 pad 11: (no net) -> GND
- U30 pad 2: (no net) -> +5V
- U30 pad 3: (no net) -> +5V
- U30 pad 4: (no net) -> unconnected-(U30-PG-Pad4)
- U30 pad 5: (no net) -> unconnected-(U30-ILIM-Pad5)
- U30 pad 6: (no net) -> unconnected-(U30-PGFB-Pad6)
- U30 pad 7: (no net) -> SET_RX1
- U30 pad 8: (no net) -> GND
- U30 pad 9: (no net) -> VCC_RX1
- U31 pad 1: (no net) -> +5V
- U31 pad 10: (no net) -> VCC_RX2
- U31 pad 11: (no net) -> GND
- U31 pad 2: (no net) -> +5V
- U31 pad 3: (no net) -> +5V
- U31 pad 4: (no net) -> unconnected-(U31-PG-Pad4)
- U31 pad 5: (no net) -> unconnected-(U31-ILIM-Pad5)
- U31 pad 6: (no net) -> unconnected-(U31-PGFB-Pad6)
- U31 pad 7: (no net) -> SET_RX2
- U31 pad 8: (no net) -> GND
- U31 pad 9: (no net) -> VCC_RX2
- U32 pad 1: (no net) -> +5V
- U32 pad 10: (no net) -> VCC_RX3
- U32 pad 11: (no net) -> GND
- U32 pad 2: (no net) -> +5V
- U32 pad 3: (no net) -> +5V
- U32 pad 4: (no net) -> unconnected-(U32-PG-Pad4)
- U32 pad 5: (no net) -> unconnected-(U32-ILIM-Pad5)
- U32 pad 6: (no net) -> unconnected-(U32-PGFB-Pad6)
- U32 pad 7: (no net) -> SET_RX3
- U32 pad 8: (no net) -> GND
- U32 pad 9: (no net) -> VCC_RX3
- U33 pad 1: (no net) -> +5V
- U33 pad 10: (no net) -> VCC_RX4
- U33 pad 11: (no net) -> GND
- U33 pad 2: (no net) -> +5V
- U33 pad 3: (no net) -> +5V
- U33 pad 4: (no net) -> unconnected-(U33-PG-Pad4)
- U33 pad 5: (no net) -> unconnected-(U33-ILIM-Pad5)
- U33 pad 6: (no net) -> unconnected-(U33-PGFB-Pad6)
- U33 pad 7: (no net) -> SET_RX4
- U33 pad 8: (no net) -> GND
- U33 pad 9: (no net) -> VCC_RX4
- U34 pad 1: (no net) -> +5V
- U34 pad 10: (no net) -> VCC_RX5
- U34 pad 11: (no net) -> GND
- U34 pad 2: (no net) -> +5V
- U34 pad 3: (no net) -> +5V
- U34 pad 4: (no net) -> unconnected-(U34-PG-Pad4)
- U34 pad 5: (no net) -> unconnected-(U34-ILIM-Pad5)
- U34 pad 6: (no net) -> unconnected-(U34-PGFB-Pad6)
- U34 pad 7: (no net) -> SET_RX5
- U34 pad 8: (no net) -> GND
- U34 pad 9: (no net) -> VCC_RX5
- U35 pad 1: (no net) -> +5V
- U35 pad 10: (no net) -> VCC_RX6
- U35 pad 11: (no net) -> GND
- U35 pad 2: (no net) -> +5V
- U35 pad 3: (no net) -> +5V
- U35 pad 4: (no net) -> unconnected-(U35-PG-Pad4)
- U35 pad 5: (no net) -> unconnected-(U35-ILIM-Pad5)
- U35 pad 6: (no net) -> unconnected-(U35-PGFB-Pad6)
- U35 pad 7: (no net) -> SET_RX6
- U35 pad 8: (no net) -> GND
- U35 pad 9: (no net) -> VCC_RX6
- U4 pad 21: (no net) -> LO_VCO_DIV
- U4 pad 3: (no net) -> +5V
- U4 pad 4: (no net) -> +5V
- U40 pad 1: (no net) -> +3V3_RF
- U40 pad 10: (no net) -> AVDD1P8_1
- U40 pad 11: (no net) -> GND
- U40 pad 2: (no net) -> +3V3_RF
- U40 pad 3: (no net) -> +3V3_RF
- U40 pad 5: (no net) -> GND
- U40 pad 8: (no net) -> REF_ADC1
- U40 pad 9: (no net) -> AVDD1P8_1
- U41 pad 1: (no net) -> +3V3_RF
- U41 pad 10: (no net) -> AVDD1P8_2
- U41 pad 11: (no net) -> GND
- U41 pad 2: (no net) -> +3V3_RF
- U41 pad 3: (no net) -> +3V3_RF
- U41 pad 5: (no net) -> GND
- U41 pad 8: (no net) -> REF_ADC2
- U41 pad 9: (no net) -> AVDD1P8_2
- U42 pad 1: (no net) -> +3V3_RF
- U42 pad 10: (no net) -> AVDD1P8_3
- U42 pad 11: (no net) -> GND
- U42 pad 2: (no net) -> +3V3_RF
- U42 pad 3: (no net) -> +3V3_RF
- U42 pad 5: (no net) -> GND
- U42 pad 8: (no net) -> REF_ADC3
- U42 pad 9: (no net) -> AVDD1P8_3
- U43 pad 1: (no net) -> +3V3_RF
- U43 pad 10: (no net) -> AVDD1P8_4
- U43 pad 11: (no net) -> GND
- U43 pad 2: (no net) -> +3V3_RF
- U43 pad 3: (no net) -> +3V3_RF
- U43 pad 5: (no net) -> GND
- U43 pad 8: (no net) -> REF_ADC4
- U43 pad 9: (no net) -> AVDD1P8_4
- U44 pad 1: (no net) -> +3V3_RF
- U44 pad 10: (no net) -> AVDD1P8_5
- U44 pad 11: (no net) -> GND
- U44 pad 2: (no net) -> +3V3_RF
- U44 pad 3: (no net) -> +3V3_RF
- U44 pad 5: (no net) -> GND
- U44 pad 8: (no net) -> REF_ADC5
- U44 pad 9: (no net) -> AVDD1P8_5
- U45 pad 1: (no net) -> +3V3_RF
- U45 pad 10: (no net) -> AVDD1P8_6
- U45 pad 11: (no net) -> GND
- U45 pad 2: (no net) -> +3V3_RF
- U45 pad 3: (no net) -> +3V3_RF
- U45 pad 5: (no net) -> GND
- U45 pad 8: (no net) -> REF_ADC6
- U45 pad 9: (no net) -> AVDD1P8_6
- U5 pad 13: (no net) -> GND
- U5 pad 15: (no net) -> GND
- U5 pad 3: (no net) -> +3V3_RF
- U5 pad 5: (no net) -> GND
- U5 pad 7: (no net) -> GND
- U50 pad 1: (no net) -> -5V_BIAS
- U50 pad 10: (no net) -> +3V3_RF
- U50 pad 11: (no net) -> +3V3_RF
- U50 pad 13: (no net) -> GND
- U50 pad 14: (no net) -> TXDRV1
- U50 pad 15: (no net) -> GND
- U50 pad 2: (no net) -> VG_PA3
- U50 pad 20: (no net) -> VG_PA1
- U50 pad 21: (no net) -> +3V3_RF
- U50 pad 22: TXDRV5 -> (no net)
- U50 pad 24: (no net) -> MCU_SPI_SCK
- U50 pad 25: (no net) -> MCU_SPI_MOSI
- U50 pad 26: (no net) -> MCU_SPI_MISO
- U50 pad 27: (no net) -> CS_BF0
- U50 pad 28: (no net) -> GND
- U50 pad 29: (no net) -> GND
- U50 pad 30: TXDRV3 -> GND
- U50 pad 31: (no net) -> TX_CHIRP
- U50 pad 32: (no net) -> GND
- U50 pad 33: (no net) -> TX_MUTE_N
- U50 pad 34: (no net) -> TX_LOAD
- U50 pad 36: (no net) -> unconnected-(U50-PA_BIAS4-Pad36)
- U50 pad 37: (no net) -> TX_MUTE_N
- U50 pad 38: TXDRV1 -> unconnected-(U50-RF4-Pad38)
- U50 pad 40: (no net) -> VG_PA5
- U50 pad 42: TX_CHIRP -> (no net)
- U50 pad 45: (no net) -> GND
- U50 pad 46: (no net) -> TXDRV5
- U50 pad 47: (no net) -> GND
- U50 pad 5: (no net) -> GND
- U50 pad 6: (no net) -> TXDRV3
- U50 pad 7: (no net) -> GND
- U51 pad 1: (no net) -> -5V_BIAS
- U51 pad 10: (no net) -> +3V3_RF
- U51 pad 11: (no net) -> +3V3_RF
- U51 pad 13: (no net) -> GND
- U51 pad 15: (no net) -> GND
- U51 pad 2: (no net) -> VG_PA4
- U51 pad 20: (no net) -> VG_PA6
- U51 pad 21: (no net) -> +3V3_RF
- U51 pad 24: (no net) -> MCU_SPI_SCK
- U51 pad 25: (no net) -> MCU_SPI_MOSI
- U51 pad 26: (no net) -> MCU_SPI_MISO
- U51 pad 27: (no net) -> CS_BF1
- U51 pad 28: (no net) -> GND
- U51 pad 29: (no net) -> GND
- U51 pad 30: (no net) -> GND
- U51 pad 31: (no net) -> TX_CHIRP
- U51 pad 32: (no net) -> GND
- U51 pad 33: (no net) -> TX_MUTE_N
- U51 pad 34: (no net) -> TX_LOAD
- U51 pad 36: (no net) -> unconnected-(U51-PA_BIAS4-Pad36)
- U51 pad 37: (no net) -> TX_MUTE_N
- U51 pad 38: (no net) -> unconnected-(U51-RF4-Pad38)
- U51 pad 40: (no net) -> VG_PA2
- U51 pad 42: TX_CHIRP -> (no net)
- U51 pad 45: (no net) -> GND
- U51 pad 47: (no net) -> GND
- U51 pad 5: (no net) -> GND
- U51 pad 7: (no net) -> GND
- U60 pad 14: (no net) -> GND
- U60 pad 15: TX1 -> TXDRV1
- U60 pad 16: (no net) -> GND
- U60 pad 18: (no net) -> VG_PA1
- U60 pad 2: (no net) -> GND
- U60 pad 21: (no net) -> PA_D1
- U60 pad 22: (no net) -> PA_D1
- U60 pad 3: TXDRV1 -> TX1
- U60 pad 4: (no net) -> GND
- U61 pad 14: (no net) -> GND
- U61 pad 16: (no net) -> GND
- U61 pad 18: (no net) -> VG_PA2
- U61 pad 2: (no net) -> GND
- U61 pad 21: (no net) -> PA_D2
- U61 pad 22: (no net) -> PA_D2
- U61 pad 4: (no net) -> GND
- U62 pad 14: (no net) -> GND
- U62 pad 15: TX3 -> TXDRV3
- U62 pad 16: (no net) -> GND
- U62 pad 18: (no net) -> VG_PA3
- U62 pad 2: (no net) -> GND
- U62 pad 21: (no net) -> PA_D3
- U62 pad 22: (no net) -> PA_D3
- U62 pad 3: TXDRV3 -> TX3
- U62 pad 4: (no net) -> GND
- U63 pad 14: (no net) -> GND
- U63 pad 16: (no net) -> GND
- U63 pad 18: (no net) -> VG_PA4
- U63 pad 2: (no net) -> GND
- U63 pad 21: (no net) -> PA_D4
- U63 pad 22: (no net) -> PA_D4
- U63 pad 4: (no net) -> GND
- U64 pad 14: (no net) -> GND
- U64 pad 15: TX5 -> TXDRV5
- U64 pad 16: (no net) -> GND
- U64 pad 18: (no net) -> VG_PA5
- U64 pad 2: (no net) -> GND
- U64 pad 21: (no net) -> PA_D5
- U64 pad 22: (no net) -> PA_D5
- U64 pad 3: TXDRV5 -> TX5
- U64 pad 4: (no net) -> GND
- U65 pad 14: (no net) -> GND
- U65 pad 16: (no net) -> GND
- U65 pad 18: (no net) -> VG_PA6
- U65 pad 2: (no net) -> GND
- U65 pad 21: (no net) -> PA_D6
- U65 pad 22: (no net) -> PA_D6
- U65 pad 4: (no net) -> GND
- U8 pad 13: (no net) -> GND
- U8 pad 15: (no net) -> GND
- U8 pad 3: (no net) -> +3V3_RF
- U8 pad 5: (no net) -> GND
- U8 pad 7: (no net) -> GND
- U9 pad 1: (no net) -> REF_100M
- U9 pad 10: (no net) -> +3V3_RF
- U9 pad 11: (no net) -> +3V3_RF
- U9 pad 12: (no net) -> +3V3_RF
- U9 pad 13: (no net) -> +3V3_RF
- U9 pad 3: (no net) -> SPI_SCLK
- U9 pad 30: (no net) -> ADC_CLK1
- U9 pad 31: (no net) -> ADC_SYSREF1
- U9 pad 32: (no net) -> ADC_CLK2
- U9 pad 33: (no net) -> ADC_SYSREF2
- U9 pad 34: (no net) -> ADC_CLK3
- U9 pad 35: (no net) -> ADC_SYSREF3
- U9 pad 36: (no net) -> ADC_CLK4
- U9 pad 37: (no net) -> ADC_SYSREF4
- U9 pad 38: (no net) -> ADC_CLK5
- U9 pad 39: (no net) -> ADC_SYSREF5
- U9 pad 4: (no net) -> CS_CLK
- U9 pad 40: (no net) -> ADC_CLK6
- U9 pad 41: (no net) -> ADC_SYSREF6
- U9 pad 42: (no net) -> FPGA_REFCLK
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Routing:
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Other:
- board text added: "10L hybrid RO4003C/RO4450F/370HR/RO4350B 2.7 mm"
- board text removed: "10L hybrid RO4003C/RO4450F/370HR/RO4350B 2.1 mm"
