File: board/kicad/HG1-PWR.kicad_pcb (KiCad board)
At the start: 6 copper layers, 146 x 30 mm, 22 parts, among them J1 M12 A-coded 8p PCB rear-mount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, J2 M12 X-coded 8p PCB rear-mount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, J3 Micro-Fit 4p to ANT: +28V_PA,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, J4 Micro-Fit 4p to DSP: +12V, J5 FFC to DSP: MDI, RS-485, 1PPS, T1 1000BASE-T magnetics (HX1188N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, U1 LT4363 surge stopper + revers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, U2 LT8640S 12 V/6 A (DSP rail), U3 LT8390 buck-boost 28 V / 1.2 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, U4 LT3462 -5 V GaN gate bias (se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, U5 LT8640S 5 V/6 A (RF rail), U6 THVD1450 RS-485 (isolated opt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

Commit message: Schematics, full-wave EM element optimisation, physical stack-ups
Schematics
- KiCad schematics for HG1-ANT/DSP/PWR generated by board/schematic/
  (33-symbol HG1 library, pins taken from the routed layout): ERC 0/0,
  schematic<->PCB parity clean; scripted "Update PCB from Schematic"
  links footprints, nets and values and stages unplaced parts.
- STM32G474 pin map corrected to the real LQFP-64 pin-out.

Full-wave EM of the radiating element (antenna/em, docs/06)
- EMerge FEM models: isolated element and infinite-array unit cell with
  a scan-matched Floquet port; local PARDISO and Modal (CPU, cuDSS GPU).
- Found and fixed: low slot/superstrate resonance of the analytic cut,
  60 deg azimuth scan blindness (element via-fence cavity), far-field
  dB scaling and E/H cut labelling.
- Differential evolution on Modal (792 solves, worst of 0/45/60 deg):
  driven 3.21 mm, parasitic 4.48 mm, slot 3.02 mm + 2.14 mm arms,
  stub 1.50 mm, 1.016 mm parasitic spacer. Active |S11| < -10 dB over
  0.52-0.70 GHz around 16 GHz at every scan to 60 az / 40 el.

Board / mechanical
- New element copper and 1,051 blind L1-L5 element-fence vias on ANT.
- Full physical stack-ups (hg1_params.STACKS) written into each
  .kicad_pcb; ANT is 2.716 mm (old 2.1 mm could not hold 10 layers).
- Enclosure, mass (1,059 g), KiCad and Blender renders regenerated.
  DRC 0 errors on all boards, parity clean.

Co-Authored-By: Claude Opus 5.5 <noreply@anthropic.com>
Parts:
- added C100: 47n, Capacitor_SMD:C_0402_1005Metric, F.Cu at (240.9, 37.5)
- added C101: 100n, Capacitor_SMD:C_0402_1005Metric, F.Cu at (246.8, 37.5)
- added C102: 1u, Capacitor_SMD:C_0402_1005Metric, F.Cu at (252.7, 37.5)
- added C103: 47u, Capacitor_SMD:C_0805_2012Metric, F.Cu at (259.3, 38.0)
- added C104: 100n, Capacitor_SMD:C_0402_1005Metric, F.Cu at (266.0, 37.5)
- added C105: 1u, Capacitor_SMD:C_0402_1005Metric, F.Cu at (271.9, 37.5)
- added C106: 4.7u, Capacitor_SMD:C_0402_1005Metric, F.Cu at (277.7, 37.5)
- added C107: 10u 50V, Capacitor_SMD:C_1210_3225Metric, F.Cu at (285.0, 38.6)
- added C108: 4.7u, Capacitor_SMD:C_0402_1005Metric, F.Cu at (292.3, 37.5)
- added CCH100: 10n 2kV, Capacitor_SMD:C_0805_2012Metric, F.Cu at (298.9, 38.0)
- added J6: Radome / board heater 10 W, Connector_JST:JST_PH_B2B-PH-K_1x02_P2.00mm_Vertical, F.Cu at (308.1, 39.8)
- added L4: 10u, Inductor_SMD:L_0805_2012Metric, F.Cu at (317.4, 37.9)
- added L5: XAL6030 2.2u, Inductor_SMD:L_Coilcraft_XAL6030-XXX, F.Cu at (326.7, 40.7)
- added Q1: N-MOSFET 80 V pass FET, Package_SO:SOIC-8_3.9x4.9mm_P1.27mm, F.Cu at (338.0, 39.8)
- added Q2: N-MOSFET 60 V, Package_SO:SOIC-8_3.9x4.9mm_P1.27mm, F.Cu at (349.4, 39.8)
- added Q3: N-MOSFET 60 V, Package_SO:SOIC-8_3.9x4.9mm_P1.27mm, F.Cu at (243.7, 51.1)
- added Q4: N-MOSFET 60 V, Package_SO:SOIC-8_3.9x4.9mm_P1.27mm, F.Cu at (255.2, 51.1)
- added Q5: N-MOSFET 60 V, Package_SO:SOIC-8_3.9x4.9mm_P1.27mm, F.Cu at (266.6, 51.1)
- added Q6: N-MOSFET heater switch, Package_SO:SOIC-8_3.9x4.9mm_P1.27mm, F.Cu at (278.1, 51.1)
- added R100: 100k, Resistor_SMD:R_0402_1005Metric, F.Cu at (286.8, 48.8)
- added R101: 10k, Resistor_SMD:R_0402_1005Metric, F.Cu at (292.7, 48.8)
- added R102: 100k, Resistor_SMD:R_0402_1005Metric, F.Cu at (298.6, 48.8)
- added R103: 2.7k, Resistor_SMD:R_0402_1005Metric, F.Cu at (304.5, 48.8)
- added R104: 100k, Resistor_SMD:R_0402_1005Metric, F.Cu at (310.4, 48.8)
- added R105: 3.3k, Resistor_SMD:R_0402_1005Metric, F.Cu at (316.3, 48.8)
- added R106: 1M, Resistor_SMD:R_0402_1005Metric, F.Cu at (322.2, 48.8)
- added R107: 73.2k, Resistor_SMD:R_0402_1005Metric, F.Cu at (328.1, 48.8)
- added R108: 18.2k, Resistor_SMD:R_0402_1005Metric, F.Cu at (334.0, 48.8)
- added R109: 1M, Resistor_SMD:R_0402_1005Metric, F.Cu at (339.9, 48.8)
- added R110: 191k, Resistor_SMD:R_0402_1005Metric, F.Cu at (345.9, 48.8)
- added R111: 18.2k, Resistor_SMD:R_0402_1005Metric, F.Cu at (351.8, 48.8)
- added R112: 4m 1%, Resistor_SMD:R_0402_1005Metric, F.Cu at (241.0, 58.4)
- added R113: 1M, Resistor_SMD:R_0402_1005Metric, F.Cu at (246.9, 58.4)
- added R114: 35.7k, Resistor_SMD:R_0402_1005Metric, F.Cu at (252.8, 58.4)
- added R115: 402k, Resistor_SMD:R_0402_1005Metric, F.Cu at (258.7, 58.4)
- added R116: 100k, Resistor_SMD:R_0402_1005Metric, F.Cu at (264.6, 58.4)
- added RCH100: 1M, Resistor_SMD:R_0402_1005Metric, F.Cu at (270.5, 58.4)
- added RHT100: 100k, Resistor_SMD:R_0402_1005Metric, F.Cu at (276.4, 58.4)
- added RS1: 5m 1%, Resistor_SMD:R_0402_1005Metric, F.Cu at (282.3, 58.4)
- added RV1: 150k, Resistor_SMD:R_0402_1005Metric, F.Cu at (288.2, 58.4)
- added RV2: 10k, Resistor_SMD:R_0402_1005Metric, F.Cu at (294.1, 58.4)
- added RV3: 100k, Resistor_SMD:R_0402_1005Metric, F.Cu at (300.1, 58.4)
- added RV4: 10k, Resistor_SMD:R_0402_1005Metric, F.Cu at (306.0, 58.4)
- added RV5: 10k, Resistor_SMD:R_0402_1005Metric, F.Cu at (311.9, 58.4)
- added RV6: 10k, Resistor_SMD:R_0402_1005Metric, F.Cu at (317.8, 58.4)
- C1: value 100 uF 50 V polymer hold-up -> 100u 50V hold-up; footprint CP_Elec_8x10 -> Capacitor_SMD:CP_Elec_8x10
- C2: value 100 uF 50 V polymer -> 100u 50V; footprint CP_Elec_8x10 -> Capacitor_SMD:CP_Elec_8x10
- D1: value SMCJ36CA TVS (MIL-STD-1275 / ISO 7637) -> SMCJ36CA; footprint D_SMC -> Diode_SMD:D_SMC
- H1, H2, H3, H4: footprint MountingHole_3.2mm_M3_Pad_Via -> MountingHole:MountingHole_3.2mm_M3_Pad_Via
- J1: value M12 A-coded 8p PCB rear-mount: 12-36 VDC, RS-485, 1PPS, discretes -> M12 A-coded 8p power/IO; footprint (none) -> HG1:M12_8P_PCB
- J2: value M12 X-coded 8p PCB rear-mount: 1000BASE-T / 2.5GBASE-T -> M12 X-coded Ethernet; footprint (none) -> HG1:M12_8P_PCB
- J3: value Micro-Fit 4p to ANT: +28V_PA, +5V -> Micro-Fit to ANT; footprint Molex_Micro-Fit_3.0_43650-0400_1x04_P3.00mm_Horizontal -> Connector_Molex:Molex_Micro-Fit_3.0_43650-0400_1x04_P3.00mm_Horizontal
- J4: value Micro-Fit 4p to DSP: +12V -> Micro-Fit to DSP; footprint Molex_Micro-Fit_3.0_43650-0400_1x04_P3.00mm_Horizontal -> Connector_Molex:Molex_Micro-Fit_3.0_43650-0400_1x04_P3.00mm_Horizontal
- J5: value FFC to DSP: MDI, RS-485, 1PPS -> FFC to DSP; footprint Hirose_FH12-30S-0.5SH_1x30-1MP_P0.50mm_Horizontal -> Connector_FFC-FPC:Hirose_FH12-30S-0.5SH_1x30-1MP_P0.50mm_Horizontal
- L1: value CM choke + DM filter (EMI, MIL-STD-461 CE102) -> DM filter 4.7u; footprint L_12x12mm_H6mm -> Inductor_SMD:L_12x12mm_H6mm
- L2: value XAL6030 4.7 uH -> XAL6030 4.7u; footprint L_Coilcraft_XAL6030-XXX -> Inductor_SMD:L_Coilcraft_XAL6030-XXX
- L3: value 10 uH 6 A shielded -> 10u 6A; footprint L_12x12mm_H6mm -> Inductor_SMD:L_12x12mm_H6mm
- T1: value 1000BASE-T magnetics (HX1188NL class) -> HX1188NL; footprint (none) -> HG1:GBE_MAG_16P
- U1: value LT4363 surge stopper + reverse-V protection -> LT4363; footprint DFN-10-1EP_3x3mm_P0.5mm_EP1.65x2.38mm -> Package_DFN_QFN:DFN-10-1EP_3x3mm_P0.5mm_EP1.65x2.38mm
- U2: value LT8640S 12 V/6 A (DSP rail) -> LT8640S 12 V; footprint QFN-24-1EP_4x4mm_P0.5mm_EP2.6x2.6mm -> Package_DFN_QFN:QFN-24-1EP_4x4mm_P0.5mm_EP2.6x2.6mm
- U3: value LT8390 buck-boost 28 V / 1.2 A GaN drain -> LT8390 28 V buck-boost; footprint QFN-28-1EP_4x5mm_P0.5mm_EP2.65x3.65mm -> Package_DFN_QFN:QFN-28-1EP_4x5mm_P0.5mm_EP2.65x3.65mm
- U4: value LT3462 -5 V GaN gate bias (sequenced) -> LT3462 -5 V; footprint TSOT-23-6 -> Package_TO_SOT_SMD:TSOT-23-6
- U5: value LT8640S 5 V/6 A (RF rail) -> LT8640S 5 V; footprint QFN-24-1EP_4x4mm_P0.5mm_EP2.6x2.6mm -> Package_DFN_QFN:QFN-24-1EP_4x4mm_P0.5mm_EP2.6x2.6mm
- U6: value THVD1450 RS-485 (isolated option) -> THVD1450; footprint SOIC-8_3.9x4.9mm_P1.27mm -> Package_SO:SOIC-8_3.9x4.9mm_P1.27mm
Connections:
- C1 pad 1: (no net) -> VIN_FILT
- C1 pad 2: (no net) -> GND
- C2 pad 1: (no net) -> +5V_RF
- C2 pad 2: (no net) -> GND
- D1 pad 1: (no net) -> VIN_RAW
- D1 pad 2: (no net) -> GND
- J1 pad 1: PWRIO_1 -> VIN_RAW
- J1 pad 2: PWRIO_2 -> VIN_RAW
- J1 pad 3: PWRIO_3 -> GND
- J1 pad 4: PWRIO_4 -> GND
- J1 pad 5: PWRIO_5 -> RS485_A
- J1 pad 6: PWRIO_6 -> RS485_B
- J1 pad 7: PWRIO_7 -> PPS_EXT
- J1 pad 8: PWRIO_8 -> DISC_IN
- J3 pad 1: (no net) -> +28V_PA
- J3 pad 2: (no net) -> +5V_RF
- J3 pad 3: (no net) -> GND
- J3 pad 4: (no net) -> GND
- J4 pad 1: (no net) -> +12V_DSP
- J4 pad 2: (no net) -> +12V_DSP
- J4 pad 3: (no net) -> GND
- J4 pad 4: (no net) -> GND
- J5 pad 1: (no net) -> PHY_MD1
- J5 pad 10: (no net) -> PHY_MD7
- J5 pad 11: (no net) -> PHY_MD8
- J5 pad 12: (no net) -> GND
- J5 pad 13: (no net) -> RS485_TX
- J5 pad 14: (no net) -> RS485_RX
- J5 pad 15: (no net) -> RS485_DE
- J5 pad 16: (no net) -> PPS_EXT
- J5 pad 17: (no net) -> DISC_IN
- J5 pad 18: (no net) -> EN_28V
- J5 pad 19: (no net) -> EN_NEG5
- J5 pad 2: (no net) -> PHY_MD2
- J5 pad 20: (no net) -> EN_RF_5V
- J5 pad 21: (no net) -> EN_HEATER
- J5 pad 22: (no net) -> VIN_SENSE
- J5 pad 23: (no net) -> V28_SENSE
- J5 pad 24: (no net) -> V5_SENSE
- J5 pad 25: (no net) -> -5V_BIAS
- J5 pad 26: (no net) -> -5V_BIAS
- J5 pad 27: (no net) -> +3V3_IO
- J5 pad 28: (no net) -> GND
- J5 pad 29: (no net) -> GND
- J5 pad 3: (no net) -> GND
- J5 pad 30: (no net) -> GND
- J5 pad 4: (no net) -> PHY_MD3
- J5 pad 5: (no net) -> PHY_MD4
- J5 pad 6: (no net) -> GND
- J5 pad 7: (no net) -> PHY_MD5
- J5 pad 8: (no net) -> PHY_MD6
- J5 pad 9: (no net) -> GND
- L1 pad 1: (no net) -> VIN_PROT
- L1 pad 2: (no net) -> VIN_FILT
- L2 pad 1: (no net) -> SW_12
- L2 pad 2: (no net) -> +12V_DSP
- L3 pad 1: (no net) -> SW1_28
- L3 pad 2: (no net) -> SW2_28
- T1 pad 1: (no net) -> PHY_MD1
- T1 pad 10: (no net) -> MDI_2
- T1 pad 11: (no net) -> MDI_3
- T1 pad 12: (no net) -> MDI_4
- T1 pad 2: (no net) -> PHY_MD2
- T1 pad 3: (no net) -> PHY_MD3
- T1 pad 4: (no net) -> PHY_MD4
- T1 pad 5: (no net) -> PHY_MD5
- T1 pad 6: (no net) -> PHY_MD6
- T1 pad 7: (no net) -> PHY_MD7
- T1 pad 8: (no net) -> PHY_MD8
- T1 pad 9: (no net) -> MDI_1
- U1 pad 1: (no net) -> VIN_RAW
- U1 pad 10: (no net) -> unconnected-(U1-FLT-Pad10)
- U1 pad 11: (no net) -> GND
- U1 pad 2: (no net) -> VIN_SNS
- U1 pad 3: (no net) -> UV_DIV
- U1 pad 4: (no net) -> OV_DIV
- U1 pad 5: (no net) -> GND
- U1 pad 6: (no net) -> SURGE_GATE
- U1 pad 7: (no net) -> VIN_PROT
- U1 pad 8: (no net) -> FB_SURGE
- U1 pad 9: (no net) -> TMR
- U2 pad 1: (no net) -> VIN_FILT
- U2 pad 10: (no net) -> SW_12
- U2 pad 11: (no net) -> SW_12
- U2 pad 12: (no net) -> unconnected-(U2-PG-Pad12)
- U2 pad 13: (no net) -> BST_12
- U2 pad 14: (no net) -> INTVCC_12
- U2 pad 17: (no net) -> GND
- U2 pad 2: (no net) -> VIN_FILT
- U2 pad 25: (no net) -> GND
- U2 pad 3: (no net) -> VIN_FILT
- U2 pad 4: (no net) -> FB_12
- U2 pad 5: (no net) -> RT_12
- U3 pad 1: (no net) -> VIN_FILT
- U3 pad 13: (no net) -> GND
- U3 pad 2: (no net) -> VIN_FILT
- U3 pad 20: (no net) -> TG1
- U3 pad 21: (no net) -> BG1
- U3 pad 22: (no net) -> TG2
- U3 pad 23: (no net) -> BG2
- U3 pad 24: (no net) -> SW1_28
- U3 pad 25: (no net) -> SW2_28
- U3 pad 26: (no net) -> unconnected-(U3-PG-Pad26)
- U3 pad 27: (no net) -> INTVCC_28
- U3 pad 29: (no net) -> GND
- U3 pad 3: (no net) -> EN_28V
- U3 pad 4: (no net) -> FB_28
- U3 pad 5: (no net) -> ISP_28
- U3 pad 6: (no net) -> +28V_PA
- U4 pad 1: (no net) -> SW_NEG
- U4 pad 2: (no net) -> GND
- U4 pad 3: (no net) -> FB_NEG
- U4 pad 4: (no net) -> EN_NEG5
- U4 pad 5: (no net) -> +5V_RF
- U4 pad 6: (no net) -> -5V_BIAS
- U5 pad 1: (no net) -> VIN_FILT
- U5 pad 10: (no net) -> SW_5
- U5 pad 11: (no net) -> SW_5
- U5 pad 12: (no net) -> unconnected-(U5-PG-Pad12)
- U5 pad 13: (no net) -> BST_5
- U5 pad 14: (no net) -> INTVCC_5
- U5 pad 17: (no net) -> GND
- U5 pad 2: (no net) -> VIN_FILT
- U5 pad 25: (no net) -> GND
- U5 pad 3: (no net) -> EN_RF_5V
- U5 pad 4: (no net) -> FB_5
- U5 pad 5: (no net) -> RT_5
- U6 pad 1: (no net) -> RS485_RX
- U6 pad 2: (no net) -> GND
- U6 pad 3: (no net) -> RS485_DE
- U6 pad 4: (no net) -> RS485_TX
- U6 pad 5: (no net) -> GND
- U6 pad 6: (no net) -> RS485_A
- U6 pad 7: (no net) -> RS485_B
- U6 pad 8: (no net) -> +3V3_IO
